File: WLED Controller.kicad_pcb (KiCad board)
At the start: 2 copper layers, 49.5 x 54 mm, 27 parts, among them J1 Conn_01x03, J2 Conn_01x03, J3 Conn_01x03, J4 Conn_01x03, J5 Conn_01x03, J6 Conn_01x03, J7 Screw_Terminal_01x02, Q1 BC547, SW1 SW_Push, U1 74125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

Commit message: Version V1.2
Uploaded old version previously
Parts:
- removed JP3, JP5: SolderJumper_3_Open, Jumper:SolderJumper-3_P1.3mm_Open_RoundedPad1.0x1.5mm
- removed JP4, JP6: SolderJumper_2_Open, Jumper:SolderJumper-2_P1.3mm_Open_RoundedPad1.0x1.5mm
- added J8: Conn_01x02, Connector_PinHeader_2.54mm:PinHeader_1x02_P2.54mm_Vertical, F.Cu at (101.1, 86.6)
- J4, J5, J6: moved to F.Cu
- JP1: value SolderJumper_3_Open -> SolderJumper_2_Open; footprint Jumper:SolderJumper-3_P1.3mm_Open_RoundedPad1.0x1.5mm -> JumpersLarge:SolderJumper-2_P3mm; moved to F.Cu
- JP2: footprint Jumper:SolderJumper-2_P1.3mm_Open_RoundedPad1.0x1.5mm -> JumpersLarge:SolderJumper-2_P3mm; moved to F.Cu
- moved SW1 38.8 mm to (102.4, 86.9)
- moved J5 37.8 mm to (137.7, 101.6), turned to 0 degrees
- moved JP1 36.0 mm to (117.5, 111.8), turned to 0 degrees
- moved JP2 33.5 mm to (114.3, 104.5), turned to 0 degrees
- moved J6 33.3 mm to (140.5, 101.6), turned to 0 degrees
- moved J4 30.1 mm to (134.9, 101.6), turned to 0 degrees
- moved U1 16.1 mm to (121.9, 69.8), turned to 0 degrees
- moved J3 0.89 mm to (130.6, 101.6)
- moved J2 0.25 mm to (128.0, 101.6)
- moved J1 0.13 mm to (125.2, 101.6)
Connections:
- J4 pad 1: Net-(J4-Pad1) -> LED5V
- J4 pad 3: Net-(J4-Pad3) -> GND
- J5 pad 1: Net-(J5-Pad1) -> LED5V
- J5 pad 3: Net-(J5-Pad3) -> GND
- J6 pad 1: Net-(J6-Pad1) -> LED5V
- J6 pad 3: Net-(J6-Pad3) -> GND
- JP1 pad 1: GND -> Net-(D2-Pad2)
- JP1 pad 2: Net-(J4-Pad3) -> +5V
- JP2 pad 1: GND -> +5V
- JP2 pad 2: Net-(J4-Pad2) -> LED5V
- U1 pad 1: GND -> +5V
- U1 pad 10: Net-(J5-Pad3) -> GND
- U1 pad 11: Net-(J6-Pad1) -> Net-(J4-Pad2)
- U1 pad 12: Net-(J6-Pad2) -> LED2OP
- U1 pad 13: Net-(J6-Pad3) -> GND
- U1 pad 2: Net-(U1-Pad2) -> GND
- U1 pad 3: Net-(J1-Pad2) -> Net-(U1-Pad3)
- U1 pad 4: Net-(J4-Pad3) -> +5V
- U1 pad 5: Net-(J4-Pad2) -> GND
- U1 pad 6: Net-(J4-Pad1) -> Net-(U1-Pad6)
- U1 pad 8: Net-(J5-Pad1) -> Net-(J1-Pad2)
- U1 pad 9: Net-(J5-Pad2) -> LED1OP
- U2 pad 11: Net-(U1-Pad2) -> LED1OP
- U2 pad 16: Net-(U2-Pad16) -> LED2OP
Routing:
- net GND: track 94.7 -> 134.8 mm
- net Net-(J4-Pad2): track 5.71 -> 29.7 mm
- net +5V: track 75.7 -> 99.6 mm
- net LED2OP: track 0.00 -> 12.1 mm
- net Net-(J8-Pad2): track 31.1 -> 42.8 mm
- net Net-(U1-Pad2): track 8.23 -> 0.00 mm
- net LED1OP: track 0.00 -> 8.04 mm
- net Net-(J4-Pad3): track 5.68 -> 0.00 mm
- net Net-(J6-Pad2): track 5.68 -> 0.00 mm
- net Net-(J5-Pad2): track 5.68 -> 0.00 mm
- net Net-(J6-Pad3): track 5.59 -> 0.00 mm
- net Net-(J5-Pad3): track 5.59 -> 0.00 mm
- net Net-(J1-Pad2): track 26.5 -> 21.7 mm
- net Net-(J6-Pad1): track 3.05 -> 0.00 mm
- net Net-(J5-Pad1): track 3.05 -> 0.00 mm
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Other:
- board text added: "J2,3,5,6 LED Power Only"
- board text added: "JP1 - Diode Bypass JP2 - Relay Bypass"
- board text added: "PIN1 (TX)"
- board text added: "PIN2 (D4)"
- board text added: "Two outputs to run 2 strips !>512 LEDs per pin. Additional pads provided for power injection."
- board text added: "V1.2"
- board text removed: "Close/Disable solder jumpers if not using direct ports J4/J5/J6 J4 - JP1&2 J5 - JP3&4 J6 - JP5&6"
- board text removed: "Din"
- board text removed: "Dout"
- board text removed: "H"
- board text removed: "J2&3 LED Power Only"
- board text removed: "J4/J5/J6"
- board text removed: "JP1/3/5"
- board text removed: "L"
- board text removed: "Solder: L = Enable H = Disable Open = J4-6"
- board text removed: "~En"
